Commit message: Add humanoid arm description package

File: humanoid_description/urdf/test_arm.urdf (robot description, URDF)
Before this commit: robot urdf_test_arm, 5 links, 4 joints
Links:
- added link base_dummy_link
Joints:
- added joint base_dummy_to_base_joint: type fixed, parent base_dummy_link, child base_link, origin xyz=0 0 0 rpy=0 0 0
