Commit message: feat(sim): add optional WBC control and headless comparison report
Add the TSID policy-impedance bridge, aligned dynamics metadata, guarded C++ enable/release, and independent viewer process. Keep the existing PD launch available and publish the English 30-trial-per-mode comparison.

Validation: 89 component tests passed; 60 valid headless ROS 2 launch trials completed. Raw logs, agent transcripts, and temporary campaign tools remain ignored.

File: humanoid_leg_description/urdf/human_offset_corrected.urdf (robot description, URDF)
Before this commit: robot ch_robot, 13 links, 12 joints
Links:
- link hip: mass 5.159055 -> 3.46458542718
- link left_foot: mass 0.765723 -> 0.592694120373
- link left_leg1: mass 2.189611 -> 1.17518545422
- link left_leg2: mass 1.709674 -> 1.67770594951
- link left_leg3: mass 3.156742 -> 1.8557940434
- link left_leg4: mass 1.980828 -> 0.977646243227
- link right_foot: mass 0.765723 -> 0.591536165263
- link right_leg1: mass 2.189548 -> 1.17908029277
- link right_leg2: mass 1.709674 -> 1.6777180051
- link right_leg3: mass 3.156742 -> 1.8443163012
- link right_leg4: mass 1.980828 -> 0.96273799775
- link torso: mass 3.175 -> 0.001
